Commit message: flc updated

File: urdf/planar2dof.urdf (robot description, URDF)
Before this commit: robot planar2dof, 5 links, 4 joints
Links:
- link planar2dof/link_striker_ee: mass 0.1 -> 0.7

Commit message: wip adrc + adrflc

File: urdf/planar2dof.urdf (robot description, URDF)
Before this commit: robot planar2dof, 5 links, 4 joints
Links:
- link planar2dof/link_striker_ee: mass 0.7 -> 0.1
